Commit message: Jazzy update and warning cleanup

File: staubli_tx2_60l_moveit_config/config/staubli_tx2_60l.ros2_control.xacro (robot description, xacro)
@@ -2,43 +2,50 @@
 <robot xmlns:xacro="http://www.ros.org/wiki/xacro">
     <xacro:macro name="staubli_tx2_60l_ros2_control" params="name initial_positions_file">
-        <xacro:property name="initial_positions" value="${load_yaml(initial_positions_file)['initial_positions']}"/>
+        <xacro:property name="initial_positions" value="${xacro.load_yaml(initial_positions_file)['initial_positions']}"/>
         <ros2_control name="${name}" type="system">
             <hardware>
-                <plugin>fake_components/GenericSystem</plugin>
+                <!-- By default, set up controllers for simulation. This won't work on real hardware -->
+                <plugin>mock_components/GenericSystem</plugin>
             </hardware>
             <joint name="joint_1">
-                <param name="initial_position">${initial_positions['joint_1']}</param>
-                <command_interface name="position" />
-                <state_interface name="position"/>
+                <command_interface name="position"/>
+                <state_interface name="position">
+                  <param name="initial_value">${initial_positions['joint_1']}</param>
+                </state_interface>
                 <state_interface name="velocity"/>
             </joint>
             <joint name="joint_2">
-                <param name="initial_position">${initial_positions['joint_2']}</param>
-                <command_interface name="position" />
-                <state_interface name="position"/>
+                <command_interface name="position"/>
+                <state_interface name="position">
+                  <param name="initial_value">${initial_positions['joint_2']}</param>
+                </state_interface>
                 <state_interface name="velocity"/>
             </joint>
             <joint name="joint_3">
-                <param name="initial_position">${initial_positions['joint_3']}</param>
-                <command_interface name="position" />
-                <state_interface name="position"/>
+                <command_interface name="position"/>
+                <state_interface name="position">
+                  <param name="initial_value">${initial_positions['joint_3']}</param>
+                </state_interface>
                 <state_interface name="velocity"/>
             </joint>
             <joint name="joint_4">
-                <param name="initial_position">${initial_positions['joint_4']}</param>
-                <command_interface name="position" />
-                <state_interface name="position"/>
+                <command_interface name="position"/>
+                <state_interface name="position">
+                  <param name="initial_value">${initial_positions['joint_4']}</param>
+                </state_interface>
                 <state_interface name="velocity"/>
             </joint>
             <joint name="joint_5">
-                <param name="initial_position">${initial_positions['joint_5']}</param>
-                <command_interface name="position" />
-                <state_interface name="position"/>
+                <command_interface name="position"/>
+                <state_interface name="position">
+                  <param name="initial_value">${initial_positions['joint_5']}</param>
+                </state_interface>
                 <state_interface name="velocity"/>
             </joint>
             <joint name="joint_6">
-                <param name="initial_position">${initial_positions['joint_6']}</param>
-                <command_interface name="position" />
-                <state_interface name="position"/>
+                <command_interface name="position"/>
+                <state_interface name="position">
+                  <param name="initial_value">${initial_positions['joint_6']}</param>
+                </state_interface>
                 <state_interface name="velocity"/>
             </joint>

File: staubli_tx2_60l_moveit_config/config/staubli_tx2_60l.urdf.xacro (robot description, xacro)
@@ -1,9 +1,9 @@
 <?xml version="1.0"?>
-<robot xmlns:xacro="http://www.ros.org/wiki/xacro" name="staubli">
+<robot xmlns:xacro="http://www.ros.org/wiki/xacro" name="staubli_tx2_60l">
     <xacro:arg name="initial_positions_file" default="initial_positions.yaml" />
-    <!-- Import panda urdf file -->
+    <!-- Import staubli_tx2_60l urdf file -->
     <xacro:include filename="$(find staubli_tx2_60l_description)/urdf/tx2_60l.xacro" />
-    <!-- Import staubli ros2_control description -->
+    <!-- Import control_xacro -->
     <xacro:include filename="staubli_tx2_60l.ros2_control.xacro" />
-    <xacro:staubli_tx2_60l_ros2_control name="StaubliTX260lFakeSystem" initial_positions_file="$(arg initial_positions_file)"/>
+    <xacro:staubli_tx2_60l_ros2_control name="FakeSystem" initial_positions_file="$(arg initial_positions_file)"/>
 </robot>
